Commit message: add robot description display launch and rviz config

File: src/diffbot_description/urdf/diffbot.urdf.xacro (robot description, xacro)
@@ -1,4 +1,4 @@
 <?xml version="1.0"?>
-<robot name="bumperbot" xmlns:xacro="http://ros.org/wiki/xacro">
+<robot name="diffbot" xmlns:xacro="http://ros.org/wiki/xacro">
   <link name="base_footprint"/>
   <link name="base_link">
@@ -55,3 +55,85 @@
     <axis xyz="0 1 0" />
   </joint>
+  <link
+    name="wheel_left_link">
+    <inertial>
+      <origin xyz="0 0.014 0" rpy="0 0 0" />
+      <mass value="0.0530086043217644" />
+      <inertia ixx="1.8792911368909E-05"  ixy="3.31256392204584E-10" ixz="-1.14082001662767E-08"
+               iyy="3.11510738759073E-05" iyz="-3.60499245082192E-10"
+               izz="1.88266886146847E-05" />
+    </inertial>
+    <visual>
+      <origin xyz="0 0 0" rpy="-1.57 0 0" />
+      <geometry>
+        <mesh filename="package://diffbot_description/meshes/wheel_left_link.STL" />
+      </geometry>
+    </visual>
+    <collision>
+      <origin xyz="0 0.015 0" rpy="-1.57 0 0" />
+      <geometry>
+        <sphere radius="0.033"/>
+      </geometry>
+    </collision>
+  </link>
+  <joint name="wheel_left_joint" type="continuous">
+    <origin xyz="0 0.0701101849418642 0" rpy="0 0 0" />
+    <parent link="base_link" />
+    <child link="wheel_left_link" />
+    <axis xyz="0 1 0" />
+  </joint>
+  <link name="caster_front_link">
+    <inertial>
+      <origin xyz="3.89968128948481E-07 2.40073004698083E-07 0.00219173397061506" rpy="0 0 0" />
+      <mass value="1.44379265037903E-06" />
+      <inertia ixx="7.23075276010246E-11" ixy="-6.10956883467859E-16" ixz="2.22849693525031E-15"
+               iyy="3.8713793085917E-11"  iyz="2.93909858781952E-15"
+               izz="1.00967486676306E-10" />
+    </inertial>
+    <visual>
+      <origin xyz="0 0 0" rpy="0 0 0" />
+      <geometry>
+        <mesh filename="package://diffbot_description/meshes/caster_front_link.STL" />
+      </geometry>
+    </visual>
+    <collision>
+      <origin xyz="0 0 0" rpy="0 0 0" />
+      <geometry>
+        <sphere radius="0.005"/>
+      </geometry>
+    </collision>
+  </link>
+  <joint name="caster_front_joint" type="fixed">
+    <origin xyz="0.04755 0 -0.0275" rpy="0 0 0" />
+    <parent link="base_link" />
+    <child link="caster_front_link" />
+    <axis xyz="0 0 0" />
+  </joint>
+  <link name="caster_rear_link">
+    <inertial>
+      <origin xyz="3.8996812895542E-07 2.40073004698083E-07 0.00219173397061509" rpy="0 0 0" />
+      <mass value="1.44379265037902E-06" />
+      <inertia ixx="7.23075276010246E-11" ixy="-6.10956872363424E-16" ixz="2.22849693527207E-15"
+               iyy="3.87137930859167E-11" iyz="2.939098587861E-15"
+               izz="1.00967486676306E-10" />
+    </inertial>
+    <visual>
+      <origin xyz="0 0 0" rpy="0 0 0" />
+      <geometry>
+        <mesh filename="package://diffbot_description/meshes/caster_rear_link.STL" />
+      </geometry>
+    </visual>
+    <collision>
+      <origin xyz="0 0 0" rpy="0 0 0" />
+      <geometry>
+        <sphere radius="0.005"/>
+      </geometry>
+    </collision>
+  </link>
+  <joint name="caster_rear_joint" type="fixed">
+    <origin xyz="-0.04755 0 -0.0275" rpy="0 0 0" />
+    <parent link="base_link" />
+    <child link="caster_rear_link" />
+    <axis xyz="0 0 0" />
+  </joint>
 </robot>

Commit message: add robot gazebo launch with materials

File: src/diffbot_description/urdf/diffbot.urdf.xacro (robot description, xacro)
@@ -1,4 +1,8 @@
 <?xml version="1.0"?>
 <robot name="diffbot" xmlns:xacro="http://ros.org/wiki/xacro">
+  <!--Gazebo Parameters -->
+  <xacro:include filename="$(find diffbot_description)/urdf/diffbot_gazebo.xacro" />
+  <!--Materials -->
+  <xacro:include filename="$(find diffbot_description)/urdf/diffbot_material.xacro" />
   <link name="base_footprint"/>
   <link name="base_link">
@@ -15,4 +19,5 @@
         <mesh filename="package://diffbot_description/meshes/base_link.STL" />
       </geometry>
+      <material name="black"/>
     </visual>
     <collision>
@@ -41,4 +46,5 @@
         <mesh filename="package://diffbot_description/meshes/wheel_right_link.STL" />
       </geometry>
+      <material name="black"/>
     </visual>
     <collision>
@@ -69,4 +75,5 @@
         <mesh filename="package://diffbot_description/meshes/wheel_left_link.STL" />
       </geometry>
+      <material name="black"/>
     </visual>
     <collision>
@@ -96,4 +103,5 @@
         <mesh filename="package://diffbot_description/meshes/caster_front_link.STL" />
       </geometry>
+      <material name="white"/>
     </visual>
     <collision>
@@ -123,4 +131,5 @@
         <mesh filename="package://diffbot_description/meshes/caster_rear_link.STL" />
       </geometry>
+      <material name="white"/>
     </visual>
     <collision>

Commit message: implement ros2 control setup

File: src/diffbot_description/urdf/diffbot.urdf.xacro (robot description, xacro)
@@ -5,4 +5,8 @@
   <!--Materials -->
   <xacro:include filename="$(find diffbot_description)/urdf/diffbot_material.xacro" />
+  <!-- Start GZ or Ignition depending on ROS 2 Version -->
+  <xacro:arg name="is_ignition" default="true"/>
+  <!-- Include ros2_control Plugins -->
+  <xacro:include filename="$(find diffbot_description)/urdf/diffbot_ros2_control.xacro" />
   <link name="base_footprint"/>
   <link name="base_link">
@@ -131,5 +135,4 @@
         <mesh filename="package://diffbot_description/meshes/caster_rear_link.STL" />
       </geometry>
-      <material name="white"/>
     </visual>
     <collision>

File: src/diffbot_description/urdf/diffbot_gazebo.xacro (robot description, xacro)
@@ -37,3 +37,24 @@
     <maxVel>1.0</maxVel>
   </gazebo>
+  <!-- ROS 2 Control: this is the Gazebo-side plugin that actually implements
+       the hardware plugin declared in diffbot_ros2_control.xacro (e.g.
+       ign_ros2_control/IgnitionSystem) — it's what connects Gazebo's physics
+       engine to ros2_control's read/write interfaces every simulation step.
+       On load, it also starts the controller_manager, which reads the YAML
+       below to know which controllers to spawn (joint_state_broadcaster,
+       velocity controller, etc). -->
+  <gazebo>
+    <!-- ROS 2 Humble -->
+    <xacro:if value="$(arg is_ignition)">
+      <plugin filename="ign_ros2_control-system" name="ign_ros2_control::IgnitionROS2ControlPlugin">
+        <parameters>$(find diffbot_controller)/config/diffbot_controllers.yaml</parameters>
+      </plugin>
+    </xacro:if>
+    <!-- ROS 2 Iron or above -->
+    <xacro:unless value="$(arg is_ignition)">
+      <plugin filename="gz_ros2_control-system" name="gz_ros2_control::GazeboSimROS2ControlPlugin">
+        <parameters>$(find diffbot_controller)/config/diffbot_controllers.yaml</parameters>
+      </plugin>
+    </xacro:unless>
+  </gazebo>
 </robot>

Commit message: create simulated noisy odometry

File: src/diffbot_description/urdf/diffbot.urdf.xacro (robot description, xacro)
@@ -94,4 +94,32 @@
     <axis xyz="0 1 0" />
   </joint>
+  <link name="imu_link">
+    <inertial>
+      <origin xyz="-0.00552433659106688 0.000168210391520346 0.000514000497342681" rpy="0 0 0" />
+      <mass value="0.000528415362211671" />
+      <inertia ixx="1.46176048428261E-08" ixy="1.40015117949421E-10" ixz="-1.99633872937403E-12"
+               iyy="8.59662482954888E-09" iyz="7.52375112767959E-12"
+               izz="2.30279421279312E-08" />
+    </inertial>
+    <visual>
+      <origin xyz="0 0 0" rpy="0 0 0" />
+      <geometry>
+        <mesh filename="package://diffbot_description/meshes/imu_link.STL" />
+      </geometry>
+      <material name="white"/>
+    </visual>
+    <collision>
+      <origin xyz="0 0 0" rpy="0 0 0" />
+      <geometry>
+        <mesh filename="package://diffbot_description/meshes/imu_link.STL" />
+      </geometry>
+    </collision>
+  </link>
+  <joint name="imu_joint" type="fixed">
+    <origin xyz="0 0 0.0698986241758014" rpy="0 0 0" />
+    <parent link="base_link" />
+    <child link="imu_link" />
+    <axis xyz="0 0 0" />
+  </joint>
   <link name="caster_front_link">
     <inertial>

File: src/diffbot_description/urdf/diffbot_gazebo.xacro (robot description, xacro)
@@ -50,4 +50,6 @@
         <parameters>$(find diffbot_controller)/config/diffbot_controllers.yaml</parameters>
       </plugin>
+      <plugin filename="ignition-gazebo-imu-system" name="ignition::gazebo::systems::Imu">
+      </plugin>
     </xacro:if>
     <!-- ROS 2 Iron or above -->
@@ -56,5 +58,58 @@
         <parameters>$(find diffbot_controller)/config/diffbot_controllers.yaml</parameters>
       </plugin>
+      <plugin filename="gz-sim-imu-system" name="gz::sim::systems::Imu">
+      </plugin>
     </xacro:unless>
   </gazebo>
+  <!-- IMU -->
+  <gazebo reference="imu_link">
+    <sensor name="imu" type="imu">
+        <always_on>true</always_on>
+        <update_rate>100</update_rate>
+        <gz_frame_id>imu_link</gz_frame_id>
+        <topic>imu</topic>
+        <imu>
+          <angular_velocity>
+            <x>
+              <noise type="gaussian">
+                <mean>0.0</mean>
+                <stddev>2e-4</stddev>
+              </noise>
+            </x>
+            <y>
+              <noise type="gaussian">
+                <mean>0.0</mean>
+                <stddev>2e-4</stddev>
+              </noise>
+            </y>
+            <z>
+              <noise type="gaussian">
+                <mean>0.0</mean>
+                <stddev>2e-4</stddev>
+              </noise>
+            </z>
+          </angular_velocity>
+          <linear_acceleration>
+            <x>
+              <noise type="gaussian">
+                <mean>0.0</mean>
+                <stddev>1.7e-2</stddev>
+              </noise>
+            </x>
+            <y>
+              <noise type="gaussian">
+                <mean>0.0</mean>
+                <stddev>1.7e-2</stddev>
+              </noise>
+            </y>
+            <z>
+              <noise type="gaussian">
+                <mean>0.0</mean>
+                <stddev>1.7e-2</stddev>
+              </noise>
+            </z>
+          </linear_acceleration>
+        </imu>
+    </sensor>
+  </gazebo>
 </robot>

Commit message: add RPLIDAR C1 2D LiDAR to diffbot

File: src/diffbot_description/urdf/diffbot.urdf.xacro (robot description, xacro)
@@ -179,3 +179,31 @@
     <axis xyz="0 0 0" />
   </joint>
+  <link name="laser_link">
+    <inertial>
+      <origin xyz="0 0 0" rpy="0 0 0" />
+      <mass value="0.073" />
+      <inertia ixx="1.96074931730795E-05" ixy="0" ixz="0"
+               iyy="2.40983835136327E-05" iyz="0"
+               izz="4.14184164228595E-05" />
+    </inertial>
+    <visual>
+      <origin xyz="0 0 0" rpy="0 0 0" />
+      <geometry>
+        <mesh filename="package://diffbot_description/meshes/laser_link.STL" />
+      </geometry>
+      <material name="dark_grey"/>
+    </visual>
+    <collision>
+      <origin xyz="0 0 0" rpy="0 0 0" />
+      <geometry>
+        <mesh filename="package://diffbot_description/meshes/laser_link.STL" />
+      </geometry>
+    </collision>
+  </link>
+  <joint name="laser_joint" type="fixed">
+    <origin xyz="-0.0050526 -0.0023221 0.1208" rpy="0 0 3.14" />
+    <parent link="base_link" />
+    <child link="laser_link" />
+    <axis xyz="0 0 0" />
+  </joint>
 </robot>

File: src/diffbot_description/urdf/diffbot_gazebo.xacro (robot description, xacro)
@@ -52,4 +52,7 @@
       <plugin filename="ignition-gazebo-imu-system" name="ignition::gazebo::systems::Imu">
       </plugin>
+      <plugin filename="ignition-gazebo-sensors-system" name="ignition::gazebo::systems::Sensors">
+        <render_engine>ogre2</render_engine>
+      </plugin>
     </xacro:if>
     <!-- ROS 2 Iron or above -->
@@ -59,4 +62,7 @@
       </plugin>
       <plugin filename="gz-sim-imu-system" name="gz::sim::systems::Imu">
+      </plugin>
+      <plugin filename="gz-sim-sensors-system" name="gz::sim::systems::Sensors">
+        <render_engine>ogre2</render_engine>
       </plugin>
     </xacro:unless>
@@ -113,3 +119,37 @@
     </sensor>
   </gazebo>
+  <!-- 2D Laser Sensor (RPLIDAR C1) -->
+  <gazebo reference="laser_link">
+    <sensor name="lidar" type="gpu_lidar">
+      <always_on>true</always_on>
+      <visualize>true</visualize>
+      <topic>scan</topic>
+      <update_rate>10</update_rate>
+      <gz_frame_id>laser_link</gz_frame_id>
+      <!-- laser_link's own origin is the mesh's bottom mounting face (z=0);
+           the RPLIDAR C1 datasheet places the actual optical window 29.8mm
+           above that, so the raycast origin is offset up to match. -->
+      <pose>0 0 0.0298 0 0 0</pose>
+      <lidar>
+        <scan>
+          <horizontal>
+            <samples>360</samples>
+            <resolution>1.00000</resolution>
+            <min_angle>0.000000</min_angle>
+            <max_angle>6.280000</max_angle>
+          </horizontal>
+        </scan>
+        <range>
+          <min>0.050000</min>
+          <max>12.0</max>
+          <resolution>0.02</resolution>
+        </range>
+        <noise>
+          <type>gaussian</type>
+          <mean>0.0</mean>
+          <stddev>0.01</stddev>
+        </noise>
+      </lidar>
+    </sensor>
+  </gazebo>
 </robot>

Commit message: adjust material urdf and laser mesh

File: src/diffbot_description/urdf/diffbot.urdf.xacro (robot description, xacro)
@@ -202,5 +202,5 @@
   </link>
   <joint name="laser_joint" type="fixed">
-    <origin xyz="-0.0050526 -0.0023221 0.1208" rpy="0 0 3.14" />
+    <origin xyz="0 0 0.0793" rpy="0 0 0" />
     <parent link="base_link" />
     <child link="laser_link" />

File: src/diffbot_description/urdf/diffbot_material.xacro (robot description, xacro)
@@ -3,4 +3,5 @@
   <xacro:property name="black_color" value="0.1 0.1 0.1 1.0" />
   <xacro:property name="white_color" value="1.0 1.0 1.0 1.0" />
+  <xacro:property name="dark_grey_color" value="0.3 0.3 0.3 1.0" />
   <material name="black">
     <color rgba="${black_color}" />
@@ -9,3 +10,6 @@
     <color rgba="${white_color}" />
   </material>
+  <material name="dark_grey">
+    <color rgba="${dark_grey_color}" />
+  </material>
 </robot>
